Commit message: ready carto to fly

File: uav_localization/urdf/uav_super.urdf (robot description, URDF)
Before this commit: robot uav_livox_tf, 3 links, 2 joints
Links:
- added link camera_init
Joints:
- added joint base_to_camera: type fixed, parent base_link, child camera_init, origin xyz=0 0.0 0.0 rpy=0 0 0
